Commit message: cara imu integrated+ behavior node run

File: ros2_ws/src/cara_motion_control/urdf/cara.urdf (robot description, URDF)
Before this commit: robot cara, 3 links, 2 joints
Links:
- added link head_link, mass 0.3; collision sphere radius=0.08; visual sphere radius=0.08
- link thigh_l: geometry collision cylinder length=0.1 radius=0.035; visual cylinder length=0.1 radius=0.035
- link torso: geometry collision box size=0.15 0.12 0.2; visual box size=0.15 0.12 0.2
Joints:
- removed joint hip_pitch_joint
- added joint hip_pitch_l: type revolute, parent torso, child thigh_l, origin xyz=0 0.08 -0.1 rpy=0 0 0, axis 0 1 0, limit lower=-1.5 upper=1.5 effort=5.0 velocity=6.0
- added joint neck_pitch: type revolute, parent torso, child head_link, origin xyz=0 0 0.18 rpy=0 0 0, axis 0 1 0, limit lower=-0.5 upper=0.5 effort=1.0 velocity=3.0
- joint base_to_torso: origin (none) -> xyz=0 0 0.1 rpy=0 0 0

File: ros2_ws/src/cara_motion_control/urdf/meshes/cara.urdf (robot description, URDF)
Before this commit: robot cara, 3 links, 2 joints
Links:
- link torso: geometry visual mesh filename=package://cara_description/meshes/torso.obj
Joints:
- joint hip_pitch_joint: limit lower=-1.0 upper=1.0 effort=2.5 velocity=6.0 -> lower=-1.57 upper=1.57 effort=2.5 velocity=6.0
